File: schematics/cpu.sch (KiCad schematic (older format))
At the start: 33 parts, among them U1 74LS86, U2 74LS86, U3 74LS283, U4 74LS283, U5 74HC245

Commit message: Started Designing the pcb for the ALU and GP registers.
Parts:
- removed SW?: SW_Push, symbol SW_Push
- added J3, J4, J5, J6: Conn_01x01, Pin_Headers:Pin_Header_Straight_1x01_Pitch2.00mm, symbol Conn_01x01
- D1, D10, D11, D12, D13, D14, D15, D16, D2, D3, D4, D5, D6, D7, D8, D9: renamed from D?; footprint (none) -> LEDs:LED_D3.0mm
- J1, J2: renamed from J?; footprint (none) -> Pin_Headers:Pin_Header_Straight_1x01_Pitch2.00mm
- U1, U2: footprint (none) -> Housings_DIP:DIP-14_W7.62mm
- U10, U11: renamed from U?; footprint (none) -> Housings_DIP:DIP-20_W7.62mm
- U12, U13, U14: renamed from U?; footprint DIP28N -> (none)
- U3, U4: footprint (none) -> Housings_DIP:DIP-16_W7.62mm
- U5: footprint (none) -> Housings_DIP:DIP-20_W7.62mm
- U6, U7, U8, U9: renamed from U?; footprint (none) -> Housings_DIP:DIP-16_W7.62mm
Connections:
- wire segments 341 -> 345
Other:
- note added: "Main Module"
- moved on the sheet: D1, D10, D11, D12, D13, D14, D15, D16, D2, D3, D4, D5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

Commit message: Finished placing tracks for the registers and ALU PCB.
Parts:
- added DATA0, DATA1, DATA3, DATA4, DATA5, DATA6, DATA7, J7: Conn_01x01, Pin_Headers:Pin_Header_Straight_1x01_Pitch2.00mm, symbol cpu-rescue:Conn_01x01
- added DATA2: (no value), Pin_Headers:Pin_Header_Straight_1x01_Pitch2.00mm, symbol cpu-rescue:Conn_01x01
- D1, D10, D11, D12, D13, D14, D15, D16, D2, D3, D4, D5, D6, D7, D8, D9: symbol LED -> cpu-rescue:LED
- J1, J2, J3, J4, J5, J6: symbol Conn_01x01 -> cpu-rescue:Conn_01x01
- U1, U2: symbol 74LS86 -> cpu-rescue:74LS86
- U10, U11, U5: symbol 74HC245 -> cpu-rescue:74HC245
- U12, U13, U14: symbol HM62256BLSP-7 -> cpu-rescue:HM62256BLSP-7
- U3, U4: symbol 74LS283 -> cpu-rescue:74LS283
- U6, U7, U8, U9: symbol 74LS173 -> cpu-rescue:74LS173
Connections:
- net labels added: VCC
- net labels removed: +5V
- wire segments 345 -> 456
